Commit message: SLAM modo Localizacion

File: description/robot_core.xacro (robot description, xacro)
@@ -36,5 +36,5 @@
     </link>
     <!-- BASE_FOOTPRINT LINK -->
-    <joint name="base_footprint_joint" type="fixed">
+    <joint name="base_footprint_joint" type="fixed">  <!-- se agrego para usar SLAM -->
         <parent link="base_link"/>
         <child link="base_footprint"/>
